File: Orthosie-Eagle-files/Orthosie.brd (EAGLE design)
At the start: 20 x 15 mm, 14 parts, among them U2 NINA-B306-00B

Commit message: Pin Correction
Parts:
- U$1: value ESP02S -> ESP02SESP02S_MIRROR; device ESP02s:ESP02S -> ESP02s:ESP02S_MIRROR
- moved U$1 3.81 mm to (1.61, 7.31)
Changed lines of the file:
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@@
 <dimension x1="0" y1="-11.75" x2="20" y2="-11.5" x3="10" y3="26.75" textsize="1.778" layer="47" dtype="horizontal"/>
 <text x="8.4" y="13.175" size="1.27" layer="25">Orthosie v2.0</text>
+<dimension x1="3.3" y1="1.9" x2="3.3" y2="1" x3="0.875" y3="1.45" textsize="1.778" layer="47" dtype="horizontal" width="0.05"/>
+<dimension x1="3" y1="2.05" x2="3.625" y2="2.1" x3="3.3125" y3="1.125" textsize="1.778" layer="47" dtype="horizontal" width="0.05"/>
 </plain>
 <attributes>
@@
 <attribute name="MF" value="U-Blox" x="12.225" y="7.525" size="1.778" layer="27" rot="R90" display="off"/>
 <attribute name="MP" value="NINA-B306-00B" x="12.225" y="7.525" size="1.778" layer="27" rot="R90" display="off"/>
-<attribute name="NAME" x="4.205" y="2.225" size="1.27" layer="25" rot="R90"/>
+<attribute name="NAME" x="6.605" y="3.075" size="1.27" layer="25" rot="R90"/>
 <attribute name="PACKAGE" value="SMD-55 U-Blox" x="12.225" y="7.525" size="1.778" layer="27" rot="R90" display="off"/>
 <attribute name="PRICE" value="None" x="12.225" y="7.525" size="1.778" layer="27" rot="R90" display="off"/>
@@
 <attribute name="VALUE" x="20.205" y="2.225" size="1.27" layer="27" rot="R90" align="top-left"/>
 </element>
-<element name="U$1" library="ESP02s" package="ESP02S" value="ESP02S" x="1.6" y="3.5" smashed="yes" rot="R90"/>
+<element name="U$1" library="ESP02s" package="ESP02S_MIRROR" value="ESP02SESP02S_MIRROR" x="1.61" y="7.31" smashed="yes" rot="R90"/>
 <element name="R1" library="Generic-0R-0402" package="RESC1005X40N" value="4.7K" x="16.1" y="1.125" smashed="yes" rot="R180">
 <attribute name="ARROW_PART_NUMBER" value="CRCW04020000Z0EE" x="16.1" y="1.125" size="1.778" layer="27" rot="R180" display="off"/>
@@
 <via x="3.5" y="10.5" extent="1-16" drill="0.1"/>
 <contactref element="U$2" pad="5"/>
-<wire x1="1.6" y1="10.5" x2="3.5" y2="10.5" width="0.254" layer="16"/>
 <via x="6.6" y="5.525" extent="1-16" drill="0.1"/>
 <via x="9.3" y="8.1" extent="1-16" drill="0.1"/>
@@
 <wire x1="11.525" y1="11.675" x2="11.525" y2="12.175" width="0.254" layer="16"/>
 <wire x1="13.15" y1="12.375" x2="14.473" y2="11.052" width="0.254" layer="16"/>
+<wire x1="3.5" y1="10.5" x2="1.61" y2="10.5" width="0.4064" layer="1"/>
 </signal>
 <signal name="SWDCLK">
@@
 <via x="12.525" y="11.675" extent="1-16" drill="0.1"/>
 <via x="3.5" y="3.5" extent="1-16" drill="0.1"/>
-<wire x1="1.6" y1="3.5" x2="3.5" y2="3.5" width="0.254" layer="1"/>
 <wire x1="11.15" y1="1.15" x2="9.66" y2="1.15" width="0.254" layer="1"/>
 <wire x1="12.525" y1="11.65" x2="12.525" y2="11.675" width="0.254" layer="1"/>
@@
 <wire x1="5.363" y1="2.262" x2="5.387" y2="2.262" width="0.2032" layer="1"/>
 <wire x1="5.387" y1="2.262" x2="5.6" y2="2.475" width="0.2032" layer="1"/>
+<wire x1="1.61" y1="3.5" x2="3.5" y2="3.5" width="0.254" layer="16"/>
 </signal>
 <signal name="MIC_PWR">
@@
 <contactref element="U2" pad="25"/>
 <via x="3.5" y="5.5" extent="1-16" drill="0.1"/>
-<wire x1="1.6" y1="5.5" x2="3.5" y2="5.5" width="0.254" layer="1"/>
 <via x="6.525" y="11.675" extent="1-16" drill="0.11"/>
 <wire x1="6.525" y1="11.65" x2="6.525" y2="11.675" width="0.254" layer="1"/>
@@
 <wire x1="6.525" y1="10.675" x2="4.775" y2="8.925" width="0.1524" layer="2"/>
 <wire x1="4.775" y1="8.925" x2="4.775" y2="6.775" width="0.1524" layer="2"/>
+<wire x1="1.61" y1="5.5" x2="3.5" y2="5.5" width="0.254" layer="16"/>
 </signal>
 <signal name="VCC">
@@
 <via x="3.5" y="12.5" extent="1-16" drill="0.1"/>
 <contactref element="U$2" pad="1"/>
-<wire x1="1.6" y1="12.5" x2="3.5" y2="12.5" width="0.4064" layer="16"/>
 <via x="14.525" y="3.375" extent="1-16" drill="0.1"/>
 <wire x1="15.525" y1="3.4" x2="15.5" y2="3.375" width="0.4064" layer="1"/>
@@
 <wire x1="18.85" y1="4.775" x2="17.45" y2="3.375" width="0.4064" layer="16"/>
 <wire x1="17.45" y1="3.375" x2="14.525" y2="3.375" width="0.4064" layer="16"/>
+<wire x1="1.61" y1="12.5" x2="3.5" y2="12.5" width="0.4064" layer="1"/>
 </signal>
 <signal name="SWDIO">
@@
 <contactref element="U$1" pad="P$3"/>
 <via x="3.5" y="7.5" extent="1-16" drill="0.1"/>
-<wire x1="1.6" y1="7.5" x2="3.5" y2="7.5" width="0.254" layer="1"/>
 <via x="11.275" y="10.275" extent="1-16" drill="0.11"/>
 <wire x1="3.5" y1="7.5" x2="4.15" y2="7.5" width="0.1524" layer="3"/>
@@
 <wire x1="4.15" y1="7.5" x2="5.6" y2="8.95" width="0.1524" layer="3"/>
 <wire x1="5.6" y1="8.95" x2="9.95" y2="8.95" width="0.1524" layer="3"/>
+<wire x1="1.61" y1="7.5" x2="3.5" y2="7.5" width="0.254" layer="16"/>
 </signal>
 <signal name="D4">
@@
 <contactref element="U$1" pad="P$5"/>
 <via x="3.5" y="11.5" extent="1-16" drill="0.1"/>
-<wire x1="1.6" y1="11.5" x2="3.5" y2="11.5" width="0.254" layer="1"/>
 <via x="10.175" y="10.275" extent="1-16" drill="0.1"/>
 <wire x1="3.5" y1="11.5" x2="4.25" y2="12.25" width="0.1524" layer="2"/>
@@
 <wire x1="4.25" y1="12.25" x2="8" y2="12.25" width="0.1524" layer="2"/>
 <wire x1="8" y1="12.25" x2="9.3" y2="10.95" width="0.1524" layer="2"/>
+<wire x1="1.61" y1="11.5" x2="3.5" y2="11.5" width="0.254" layer="16"/>
 </signal>
 <signal name="D5">
@@
 <contactref element="U$1" pad="P$6"/>
 <via x="3.5" y="2.5" extent="1-16" drill="0.1"/>
-<wire x1="1.6" y1="2.5" x2="3.5" y2="2.5" width="0.254" layer="16"/>
 <via x="9.525" y="11.65" extent="1-16" drill="0.11"/>
 <wire x1="9.525" y1="11.65" x2="7.875" y2="11.65" width="0.1524" layer="15"/>
@@
 <wire x1="7.875" y1="11.65" x2="4.7" y2="8.475" width="0.1524" layer="15"/>
 <wire x1="4.7" y1="8.475" x2="4.7" y2="3.7" width="0.1524" layer="15"/>
+<wire x1="1.61" y1="2.5" x2="3.5" y2="2.5" width="0.254" layer="1"/>
 </signal>
 <signal name="D3">
@@
 <contactref element="U$1" pad="P$4"/>
 <via x="3.5" y="9.5" extent="1-16" drill="0.1"/>
-<wire x1="1.6" y1="9.5" x2="3.5" y2="9.5" width="0.254" layer="1"/>
 <via x="10.5" y="11.65" extent="1-16" drill="0.11"/>
 <wire x1="10.525" y1="11.65" x2="10.5" y2="11.65" width="0.254" layer="1"/>
@@
 <wire x1="5.55" y1="9.5" x2="7.075" y2="11.025" width="0.1524" layer="14"/>
 <wire x1="7.075" y1="11.025" x2="9.875" y2="11.025" width="0.1524" layer="14"/>
+<wire x1="1.61" y1="9.5" x2="3.5" y2="9.5" width="0.254" layer="16"/>
 </signal>
 <signal name="D6">
@@
 <contactref element="U$1" pad="P$7"/>
 <via x="3.5" y="4.5" extent="1-16" drill="0.1"/>
-<wire x1="1.6" y1="4.5" x2="3.5" y2="4.5" width="0.254" layer="16"/>
 <via x="9.075" y="10.275" extent="1-16" drill="0.11"/>
 <wire x1="3.5" y1="4.5" x2="9.075" y2="10.075" width="0.1524" layer="2"/>
 <wire x1="9.075" y1="10.075" x2="9.075" y2="10.275" width="0.1524" layer="2"/>
+<wire x1="1.61" y1="4.5" x2="3.5" y2="4.5" width="0.254" layer="1"/>
 </signal>
 <signal name="D7">
@@
 <contactref element="U$1" pad="P$8"/>
 <via x="3.5" y="6.5" extent="1-16" drill="0.1"/>
-<wire x1="1.6" y1="6.5" x2="3.5" y2="6.5" width="0.254" layer="16"/>
 <via x="5.4" y="11.55" extent="1-16" drill="0.11"/>
 <wire x1="5.375" y1="11.525" x2="5.4" y2="11.55" width="0.254" layer="1"/>
@@
 <wire x1="4.425" y1="7.425" x2="3.5" y2="6.5" width="0.1524" layer="2"/>
 <wire x1="4.425" y1="10.575" x2="4.425" y2="7.425" width="0.1524" layer="2"/>
+<wire x1="1.61" y1="6.5" x2="3.5" y2="6.5" width="0.254" layer="1"/>
 </signal>
 <signal name="D8">
@@
 <contactref element="U$1" pad="P$9"/>
 <via x="3.5" y="8.5" extent="1-16" drill="0.1"/>
-<wire x1="1.6" y1="8.5" x2="3.5" y2="8.5" width="0.254" layer="16"/>
 <via x="5.375" y="10.55" extent="1-16" drill="0.11"/>
 <wire x1="5.375" y1="10.525" x2="5.375" y2="10.55" width="0.254" layer="1"/>
@@
 <wire x1="5.375" y1="9.325" x2="5.375" y2="10.55" width="0.1524" layer="3"/>
 <wire x1="4.55" y1="8.5" x2="5.375" y2="9.325" width="0.1524" layer="3"/>
+<wire x1="1.61" y1="8.5" x2="3.5" y2="8.5" width="0.254" layer="1"/>
 </signal>
 <signal name="VBUS">
